File: weather_external.sch (KiCad schematic (older format))
At the start: 31 parts, among them J1 Conn_01x02_Male, J2 USB_B_Mini, J3 Conn_01x02_Male, J4 Conn_01x02_Male, J8 FTDI, Q1 DMG2305UX-13, SW1 SW_Push, U1 MCP73831-2-OT, U2 MCP1700T-3302E_TT

Commit message: V1.5 removing battery charger components
Parts:
- removed C4, C7: CP, Capacitor_THT:CP_Radial_D4.0mm_P1.50mm, symbol Device:CP
- removed D1: GREEN, LED_SMD:LED_1206_3216Metric, symbol Device:LED
- removed D2: RED, LED_SMD:LED_1206_3216Metric, symbol Device:LED
- removed D3: 1N4148, Diode_THT:D_T-1_P5.08mm_Horizontal, symbol Device:D
- removed J1: Conn_01x02_Male, Connector_Wire:SolderWire-0.1sqmm_1x02_P3.6mm_D0.4mm_OD1mm, symbol Connector:Conn_01x02_Male
- removed Q1: DMG2305UX-13, digikey-footprints:SOT-23-3, symbol dk_Transistors-FETs-MOSFETs-Single:DMG2305UX-13
- removed R5, R6: 220, Resistor_SMD:R_1206_3216Metric_Pad1.42x1.75mm_HandSolder, symbol Device:R_Small
- removed R7: 2k, Resistor_SMD:R_1206_3216Metric_Pad1.42x1.75mm_HandSolder, symbol Device:R_Small
- removed R8: 100k, Resistor_SMD:R_1206_3216Metric_Pad1.42x1.75mm_HandSolder, symbol Device:R_Small
- removed U1: MCP73831-2-OT, Package_TO_SOT_SMD:SOT-23-5, symbol Battery_Management:MCP73831-2-OT
Connections:
- net labels removed: VBAT
- wire segments 111 -> 71

Commit message: V 1.5 - no load management once it is built to run in solar panel charging mode
Parts:
- removed C1: 0.1uf, Capacitor_THT:CP_Radial_D4.0mm_P1.50mm, symbol Device:C
- removed C2: 47uf, Capacitor_THT:CP_Radial_D4.0mm_P1.50mm, symbol Device:C
- removed D4: 1N4148, Diode_THT:D_T-1_P5.08mm_Horizontal, symbol Device:D
- added C4, C7: CP, Capacitor_THT:CP_Radial_D4.0mm_P1.50mm, symbol Device:CP
- added D1: GREEN, LED_SMD:LED_1206_3216Metric, symbol Device:LED
- added D2: RED, LED_SMD:LED_1206_3216Metric, symbol Device:LED
- added J1: Battery, Connector_Wire:SolderWire-0.1sqmm_1x02_P3.6mm_D0.4mm_OD1mm, symbol Connector:Conn_01x02_Male
- added R5, R6: 220, Resistor_SMD:R_1206_3216Metric_Pad1.42x1.75mm_HandSolder, symbol Device:R_Small
- added R7: 2k, Resistor_SMD:R_1206_3216Metric_Pad1.42x1.75mm_HandSolder, symbol Device:R_Small
- added U1: MCP73831-2-OT, Package_TO_SOT_SMD:SOT-23-5, symbol Battery_Management:MCP73831-2-OT
- J3: value Conn_01x02_Male -> Solar Panel
Connections:
- net labels added: +5V, VBAT
- wire segments 71 -> 92
Other:
- moved on the sheet: J3, J8
